File: modules/higgs/hardware/higgs.sch (KiCad schematic (older format))
At the start: 4 parts

Commit message: wip: higgs schematic
Parts:
- removed C?: C_Small, symbol Device:C_Small
- removed U?: STM32F303RETx, Package_QFP:LQFP-64_10x10mm_P0.5mm, symbol MCU_ST_STM32F3:STM32F303RETx
Connections:
- no-connect marks 25 -> 0
Other:
- note removed: "TODO: \n"
- note removed: "TODO: for debugger printf, could be useful\n"
- moved on the sheet: R?, SW?
