File: modules/higgs/hardware/_autosave-higgs.kicad_pcb (KiCad board)
At the start: 2 copper layers, 2 parts, among them U1 V7803-500

Commit message: wip: modules/higgs/hardware
Parts:
- added C1: 25V 22uF, Capacitor_SMD:C_1206_3216Metric_Pad1.33x1.80mm_HandSolder, F.Cu at (51.4, -15.1)
- added C2: 25V 22uF, Capacitor_SMD:C_1206_3216Metric_Pad1.33x1.80mm_HandSolder, F.Cu at (51.4, -11.7)
- added C3: 25V 22uF, Capacitor_SMD:C_1206_3216Metric_Pad1.33x1.80mm_HandSolder, F.Cu at (61.2, -23.3)
- added C4: 25V 22uF, Capacitor_SMD:C_1206_3216Metric_Pad1.33x1.80mm_HandSolder, F.Cu at (57.4, -15.1)
- added D1: 40V 600mV@1A 1A, Diode_SMD:D_SOD-123, F.Cu at (61.1, -20.0)
- added D2: 40V 600mV@1A 1A, Diode_SMD:D_SOD-123, F.Cu at (67.1, -23.3)
- added J1: PinHeader_2x05_P2.54mm_Vertical, Connector_PinHeader_2.54mm:PinHeader_2x05_P2.54mm_Vertical, F.Cu at (43.5, -22.7)
- added L1: 100Ω@100MHz, Inductor_SMD:L_0805_2012Metric_Pad1.15x1.40mm_HandSolder, F.Cu at (56.8, -11.9)
- added L2: 100Ω@100MHz, Inductor_SMD:L_0805_2012Metric_Pad1.15x1.40mm_HandSolder, F.Cu at (62.8, -16.8)
- added L3: 100Ω@100MHz, Inductor_SMD:L_0805_2012Metric_Pad1.15x1.40mm_HandSolder, F.Cu at (66.3, -20.2)
- added U2: AMS1117-3.3, Package_TO_SOT_SMD:SOT-223-3_TabPin2, F.Cu at (53.3, -20.9)
- added U3: STM32F303RETx, Package_QFP:LQFP-64_10x10mm_P0.5mm, F.Cu at (81.3, -17.8)
- C3: value 25V 10uF -> 25V 22uF ±10%
Other:
- net class Default removed
